Commit message: Add stl file

File: slides/ros-model-display/code/ros2/ur5e_with_eef.xacro (robot description, xacro)
@@ -13,5 +13,5 @@
             <origin xyz="0 0 0.0001" rpy="0 0 0" />
             <geometry>
-                <mesh filename="package://grinding_descriptions/mesh/end_effector/pestle_ur.stl" />
+                <mesh filename="package://ros_study/meshes/pestle_ur.stl" />
             </geometry>
         </visual>
@@ -19,5 +19,5 @@
             <origin xyz="0 0 0.0001" rpy="0 0 0" />
             <geometry>
-                <mesh filename="package://grinding_descriptions/mesh/end_effector/pestle_ur.stl" />
+                <mesh filename="package://ros_study/meshes/pestle_ur.stl" />
             </geometry>
         </collision>
@@ -37,5 +37,5 @@
             <origin xyz="0 0 0.0001" rpy="0 0 0" />
             <geometry>
-                <mesh filename="package://grinding_descriptions/mesh/end_effector/spatula.stl" />
+                <mesh filename="package://ros_study/mesh/end_effector/spatula.stl" />
             </geometry>
         </visual>
@@ -43,5 +43,5 @@
             <origin xyz="0 0 0.0001" rpy="0 0 0" />
             <geometry>
-                <mesh filename="package://grinding_descriptions/mesh/end_effector/spatula.stl" />
+                <mesh filename="package://ros_study/mesh/end_effector/spatula.stl" />
             </geometry>
         </collision>

Commit message: Fix path

File: slides/ros-model-display/code/ros2/ur5e_with_eef.xacro (robot description, xacro)
@@ -37,5 +37,5 @@
             <origin xyz="0 0 0.0001" rpy="0 0 0" />
             <geometry>
-                <mesh filename="package://ros_study/mesh/end_effector/spatula.stl" />
+                <mesh filename="package://ros_study/meshes/spatula.stl" />
             </geometry>
         </visual>
@@ -43,5 +43,5 @@
             <origin xyz="0 0 0.0001" rpy="0 0 0" />
             <geometry>
-                <mesh filename="package://ros_study/mesh/end_effector/spatula.stl" />
+                <mesh filename="package://ros_study/meshes/spatula.stl" />
             </geometry>
         </collision>
