Commit message: Fix xacro

File: slides/ros-model-display/code/ros2/ur5e.xacro (robot description, xacro)
@@ -1,15 +1,13 @@
 <?xml version="1.0"?>
 <robot name="ur5e_robot" xmlns:xacro="http://ros.org/wiki/xacro">
-  <xacro:property name="DEG_TO_RAD" value="0.017453292519943295"/>
-  <xacro:property name="PI" value="3.14159265359"/>
-  <xacro:property name="PI_2" value="${PI / 2}"/>
-  <xacro:property name="PI_4" value="${PI / 4}"/>
+  <xacro:property name="mesh_visual_path" value="package://ur_description/meshes/ur5e/visual"/>
+  <xacro:property name="mesh_collision_path" value="package://ur_description/meshes/ur5e/collision"/>
   <material name="LightGrey">
     <color rgba="0.7 0.7 0.7 1.0"/>
   </material>
-  <xacro:macro name="standard_link" params="name mass ixx iyy izz ixy ixz iyz *visual_origin *collision_origin *inertial_origin visual_mesh collision_mesh">
+  <xacro:macro name="standard_link" params="name mass ixx iyy izz ixy ixz iyz visual_mesh collision_mesh visual_xyz visual_rpy collision_xyz collision_rpy inertial_xyz inertial_rpy">
     <link name="${name}">
       <visual>
-        <xacro:insert_block name="visual_origin" />
+        <origin xyz="${visual_xyz}" rpy="${visual_rpy}"/>
         <geometry>
           <mesh filename="${visual_mesh}"/>
@@ -18,5 +16,5 @@
       </visual>
       <collision>
-        <xacro:insert_block name="collision_origin" />
+        <origin xyz="${collision_xyz}" rpy="${collision_rpy}"/>
         <geometry>
           <mesh filename="${collision_mesh}"/>
@@ -25,5 +23,5 @@
       <inertial>
         <mass value="${mass}"/>
-        <xacro:insert_block name="inertial_origin" />
+        <origin xyz="${inertial_xyz}" rpy="${inertial_rpy}"/>
         <inertia ixx="${ixx}" ixy="${ixy}" ixz="${ixz}" iyy="${iyy}" iyz="${iyz}" izz="${izz}"/>
       </inertial>
@@ -50,78 +48,71 @@
     name="base_link"
     mass="4.0"
-    ixx="0.00443333156" iyy="0.00443333156" izz="0.0072"
-    ixy="0.0" ixz="0.0" iyz="0.0"
-    visual_mesh="package://ur_description/meshes/ur5e/visual/base.dae"
-    collision_mesh="package://ur_description/meshes/ur5e/collision/base.stl">
-    <visual_origin rpy="0 0 ${PI}" xyz="0 0 0"/>
-    <collision_origin rpy="0 0 ${PI}" xyz="0 0 0"/>
-    <inertial_origin rpy="0 0 0" xyz="0.0 0.0 0.0"/>
-  </xacro:standard_link>
+    ixx="0.00443333156" iyy="0.00443333156" izz="0.0072" ixy="0.0" ixz="0.0" iyz="0.0"
+    visual_mesh="${mesh_visual_path}/base.dae" collision_mesh="${mesh_collision_path}/base.stl"
+    visual_xyz="0 0 0" visual_rpy="0 0 ${pi}"
+    collision_xyz="0 0 0" collision_rpy="0 0 ${pi}"
+    inertial_xyz="0 0 0" inertial_rpy="0 0 0"
+  />
+  <xacro:revolute_joint name="shoulder_pan_joint" parent="base_link" child="shoulder_link" origin_xyz="0 0 0.1625" origin_rpy="0 0 ${pi}" axis_xyz="0 0 1" effort="150.0" lower_limit="${-pi}" upper_limit="${pi}" velocity="${pi}" damping="0.0" friction="0.0"/>
   <xacro:standard_link
     name="shoulder_link"
     mass="3.7"
-    ixx="0.010267495893" iyy="0.010267495893" izz="0.00666"
-    ixy="0.0" ixz="0.0" iyz="0.0"
-    visual_mesh="package://ur_description/meshes/ur5e/visual/shoulder.dae"
-    collision_mesh="package://ur_description/meshes/ur5e/collision/shoulder.stl">
-    <visual_origin rpy="0 0 ${PI}" xyz="0 0 0"/>
-    <collision_origin rpy="0 0 ${PI}" xyz="0 0 0"/>
-    <inertial_origin rpy="0 0 0" xyz="0.0 0.0 0.0"/>
-  </xacro:standard_link>
+    ixx="0.010267495893" iyy="0.010267495893" izz="0.00666" ixy="0.0" ixz="0.0" iyz="0.0"
+    visual_mesh="${mesh_visual_path}/shoulder.dae" collision_mesh="${mesh_collision_path}/shoulder.stl"
+    visual_xyz="0 0 0" visual_rpy="0 0 ${pi}"
+    collision_xyz="0 0 0" collision_rpy="0 0 ${pi}"
+    inertial_xyz="0 0 0" inertial_rpy="0 0 0"
+  />
+  <xacro:revolute_joint name="shoulder_lift_joint" parent="shoulder_link" child="upper_arm_link" origin_xyz="0 0 0" origin_rpy="${pi/2} 0 0" axis_xyz="0 0 1" effort="150.0" lower_limit="${-pi}" upper_limit="${pi}" velocity="${pi}" damping="0.0" friction="0.0"/>
   <xacro:standard_link
     name="upper_arm_link"
     mass="8.393"
-    ixx="0.138134736413" iyy="0.138134736413" izz="0.0236053125"
-    ixy="0.0" ixz="0.0" iyz="0.0"
-    visual_mesh="package://ur_description/meshes/ur5e/visual/upperarm.dae"
-    collision_mesh="package://ur_description/meshes/ur5e/collision/upperarm.stl">
-    <visual_origin rpy="${PI_2} 0 ${-PI_2}" xyz="0 0 0.138"/>
-    <collision_origin rpy="${PI_2} 0 ${-PI_2}" xyz="0 0 0.138"/>
-    <inertial_origin rpy="0 ${PI_2} 0" xyz="-0.2125 0.0 0.138"/>
-  </xacro:standard_link>
+    ixx="0.138134736413" iyy="0.138134736413" izz="0.0236053125" ixy="0.0" ixz="0.0" iyz="0.0"
+    visual_mesh="${mesh_visual_path}/upperarm.dae" collision_mesh="${mesh_collision_path}/upperarm.stl"
+    visual_xyz="0 0 0.138" visual_rpy="${pi/2} 0 ${-pi/2}"
+    collision_xyz="0 0 0.138" collision_rpy="${pi/2} 0 ${-pi/2}"
+    inertial_xyz="-0.2125 0.0 0.138" inertial_rpy="0 ${pi/2} 0"
+  />
+  <xacro:revolute_joint name="elbow_joint" parent="upper_arm_link" child="forearm_link" origin_xyz="-0.425 0 0" origin_rpy="0 0 0" axis_xyz="0 0 1" effort="150.0" lower_limit="${-pi}" upper_limit="${pi}" velocity="${pi}" damping="0.0" friction="0.0"/>
   <xacro:standard_link
     name="forearm_link"
     mass="2.275"
-    ixx="0.0323610733889" iyy="0.0323610733889" izz="0.0063984375"
-    ixy="0.0" ixz="0.0" iyz="0.0"
-    visual_mesh="package://ur_description/meshes/ur5e/visual/forearm.dae"
-    collision_mesh="package://ur_description/meshes/ur5e/collision/forearm.stl">
-    <visual_origin rpy="${PI_2} 0 ${-PI_2}" xyz="0 0 0.007"/>
-    <collision_origin rpy="${PI_2} 0 ${-PI_2}" xyz="0 0 0.007"/>
-    <inertial_origin rpy="0 ${PI_2} 0" xyz="-0.2125 0.0 0.007"/>
-  </xacro:standard_link>
+    ixx="0.0323610733889" iyy="0.0323610733889" izz="0.0063984375" ixy="0.0" ixz="0.0" iyz="0.0"
+    visual_mesh="${mesh_visual_path}/forearm.dae" collision_mesh="${mesh_collision_path}/forearm.stl"
+    visual_xyz="0 0 0.007" visual_rpy="${pi/2} 0 ${-pi/2}"
+    collision_xyz="0 0 0.007" collision_rpy="${pi/2} 0 ${-pi/2}"
+    inertial_xyz="-0.2125 0.0 0.007" inertial_rpy="0 ${pi/2} 0"
+  />
+  <xacro:revolute_joint name="wrist_1_joint" parent="forearm_link" child="wrist_1_link" origin_xyz="-0.3922 0 0.1333" origin_rpy="0 0 0" axis_xyz="0 0 1" effort="28.0" lower_limit="${-pi}" upper_limit="${pi}" velocity="${2*pi}" damping="0.0" friction="0.0"/>
   <xacro:standard_link
     name="wrist_1_link"
     mass="1.219"
-    ixx="0.00272396513625" iyy="0.00272396513625" izz="0.0034284375"
-    ixy="0.0" ixz="0.0" iyz="0.0"
-    visual_mesh="package://ur_description/meshes/ur5e/visual/wrist1.dae"
-    collision_mesh="package://ur_description/meshes/ur5e/collision/wrist1.stl">
-    <visual_origin rpy="${PI_2} 0 0" xyz="0 0 -0.127"/>
-    <collision_origin rpy="${PI_2} 0 0" xyz="0 0 -0.127"/>
-    <inertial_origin rpy="0 0 0" xyz="0.0 0.0 0.0"/>
-  </xacro:standard_link>
+    ixx="0.00272396513625" iyy="0.00272396513625" izz="0.0034284375" ixy="0.0" ixz="0.0" iyz="0.0"
+    visual_mesh="${mesh_visual_path}/wrist1.dae" collision_mesh="${mesh_collision_path}/wrist1.stl"
+    visual_xyz="0 0 -0.127" visual_rpy="${pi/2} 0 0"
+    collision_xyz="0 0 -0.127" collision_rpy="${pi/2} 0 0"
+    inertial_xyz="0 0 0" inertial_rpy="0 0 0"
+  />
+  <xacro:revolute_joint name="wrist_2_joint" parent="wrist_1_link" child="wrist_2_link" origin_xyz="0 -0.0997 -2.0448811823e-11" origin_rpy="${pi/2} 0 0" axis_xyz="0 0 1" effort="28.0" lower_limit="${-pi}" upper_limit="${pi}" velocity="${2*pi}" damping="0.0" friction="0.0"/>
   <xacro:standard_link
     name="wrist_2_link"
     mass="1.219"
-    ixx="0.00272194058122" iyy="0.00272194058122" izz="0.0034284375"
-    ixy="0.0" ixz="0.0" iyz="0.0"
-    visual_mesh="package://ur_description/meshes/ur5e/visual/wrist2.dae"
-    collision_mesh="package://ur_description/meshes/ur5e/collision/wrist2.stl">
-    <visual_origin rpy="0 0 0" xyz="0 0 -0.0997"/>
-    <collision_origin rpy="0 0 0" xyz="0 0 -0.0997"/>
-    <inertial_origin rpy="0 0 0" xyz="0.0 0.0 0.0"/>
-  </xacro:standard_link>
+    ixx="0.00272194058122" iyy="0.00272194058122" izz="0.0034284375" ixy="0.0" ixz="0.0" iyz="0.0"
+    visual_mesh="${mesh_visual_path}/wrist2.dae" collision_mesh="${mesh_collision_path}/wrist2.stl"
+    visual_xyz="0 0 -0.0997" visual_rpy="0 0 0"
+    collision_xyz="0 0 -0.0997" collision_rpy="0 0 0"
+    inertial_xyz="0 0 0" inertial_rpy="0 0 0"
+  />
+  <xacro:revolute_joint name="wrist_3_joint" parent="wrist_2_link" child="wrist_3_link" origin_xyz="0 0.0996 -2.04283014801e-11" origin_rpy="${pi/2} ${pi} ${pi}" axis_xyz="0 0 1" effort="28.0" lower_limit="${-pi}" upper_limit="${pi}" velocity="${2*pi}" damping="0.0" friction="0.0"/>
   <xacro:standard_link
     name="wrist_3_link"
     mass="0.1879"
-    ixx="0.000134270154625" iyy="0.000134270154625" izz="0.00019024875"
-    ixy="0.0" ixz="0.0" iyz="0.0"
-    visual_mesh="package://ur_description/meshes/ur5e/visual/wrist3.dae"
-    collision_mesh="package://ur_description/meshes/ur5e/collision/wrist3.stl">
-    <visual_origin rpy="${PI_2} 0 0" xyz="0 0 -0.0989"/>
-    <collision_origin rpy="${PI_2} 0 0" xyz="0 0 -0.0989"/>
-    <inertial_origin rpy="0 0 0" xyz="0.0 0.0 -0.025"/>
-  </xacro:standard_link>
+    ixx="0.000134270154625" iyy="0.000134270154625" izz="0.00019024875" ixy="0.0" ixz="0.0" iyz="0.0"
+    visual_mesh="${mesh_visual_path}/wrist3.dae" collision_mesh="${mesh_collision_path}/wrist3.stl"
+    visual_xyz="0 0 -0.0989" visual_rpy="${pi/2} 0 0"
+    collision_xyz="0 0 -0.0989" collision_rpy="${pi/2} 0 0"
+    inertial_xyz="0 0 -0.025" inertial_rpy="0 0 0"
+  />
+  <xacro:fixed_joint name="ee_fixed_joint" parent="wrist_3_link" child="ee_link" origin_xyz="0.0 0.0 0.0" origin_rpy="0.0 ${-pi/2} ${pi/2}"/>
   <link name="ee_link">
     <collision>
@@ -133,107 +124,6 @@
   </link>
   <link name="base"/>
+  <xacro:fixed_joint name="base_link-base_fixed_joint" parent="base_link" child="base" origin_xyz="0 0 0" origin_rpy="0 0 ${-pi}"/>
   <link name="tool0"/>
-  <link name="world"/>
-  <xacro:revolute_joint
-    name="shoulder_pan_joint"
-    parent="base_link"
-    child="shoulder_link"
-    origin_xyz="0 0 0.1625"
-    origin_rpy="0 0 ${PI}"
-    axis_xyz="0 0 1"
-    effort="150.0"
-    lower_limit="${-PI}"
-    upper_limit="${PI}"
-    velocity="${PI}"
-    damping="0.0"
-    friction="0.0"/>
-  <xacro:revolute_joint
-    name="shoulder_lift_joint"
-    parent="shoulder_link"
-    child="upper_arm_link"
-    origin_xyz="0 0 0"
-    origin_rpy="${PI_2} 0 0"
-    axis_xyz="0 0 1"
-    effort="150.0"
-    lower_limit="${-PI}"
-    upper_limit="${PI}"
-    velocity="${PI}"
-    damping="0.0"
-    friction="0.0"/>
-  <xacro:revolute_joint
-    name="elbow_joint"
-    parent="upper_arm_link"
-    child="forearm_link"
-    origin_xyz="-0.425 0 0"
-    origin_rpy="0 0 0"
-    axis_xyz="0 0 1"
-    effort="150.0"
-    lower_limit="${-PI}"
-    upper_limit="${PI}"
-    velocity="${PI}"
-    damping="0.0"
-    friction="0.0"/>
-  <xacro:revolute_joint
-    name="wrist_1_joint"
-    parent="forearm_link"
-    child="wrist_1_link"
-    origin_xyz="-0.3922 0 0.1333"
-    origin_rpy="0 0 0"
-    axis_xyz="0 0 1"
-    effort="28.0"
-    lower_limit="${-PI}"
-    upper_limit="${PI}"
-    velocity="${2 * PI}"
-    damping="0.0"
-    friction="0.0"/>
-  <xacro:revolute_joint
-    name="wrist_2_joint"
-    parent="wrist_1_link"
-    child="wrist_2_link"
-    origin_xyz="0 -0.0997 -2.0448811823e-11"
-    origin_rpy="${PI_2} 0 0"
-    axis_xyz="0 0 1"
-    effort="28.0"
-    lower_limit="${-PI}"
-    upper_limit="${PI}"
-    velocity="${2 * PI}"
-    damping="0.0"
-    friction="0.0"/>
-  <xacro:revolute_joint
-    name="wrist_3_joint"
-    parent="wrist_2_link"
-    child="wrist_3_link"
-    origin_xyz="0 0.0996 -2.04283014801e-11"
-    origin_rpy="${PI_2} ${PI} ${PI}"
-    axis_xyz="0 0 1"
-    effort="28.0"
-    lower_limit="${-PI}"
-    upper_limit="${PI}"
-    velocity="${2 * PI}"
-    damping="0.0"
-    friction="0.0"/>
-  <xacro:fixed_joint
-    name="ee_fixed_joint"
-    parent="wrist_3_link"
-    child="ee_link"
-    origin_xyz="0.0 0.0 0.0"
-    origin_rpy="0.0 ${-PI_2} ${PI_2}"/>
-  <xacro:fixed_joint
-    name="base_link-base_fixed_joint"
-    parent="base_link"
-    child="base"
-    origin_xyz="0 0 0"
-    origin_rpy="0 0 ${-PI}"/>
-  <xacro:fixed_joint
-    name="wrist_3_link-tool0_fixed_joint"
-    parent="wrist_3_link"
-    child="tool0"
-    origin_xyz="0 0 0"
-    origin_rpy="0 0 0"/>
-  <xacro:fixed_joint
-    name="world_joint"
-    parent="world"
-    child="base_link"
-    origin_xyz="0.0 0.0 0.0"
-    origin_rpy="0.0 0.0 0.0"/>
-</robot>
+  <xacro:fixed_joint name="wrist_3_link-tool0_fixed_joint" parent="wrist_3_link" child="tool0" origin_xyz="0 0 0" origin_rpy="0 0 0"/>
+  </robot>

File: slides/ros-model-display/code/ros2/ur5e_with_eef.xacro (robot description, xacro)
@@ -7,5 +7,6 @@
     <joint name="world_joint" type="fixed">
         <parent link="world" />
-        <child link="base_link" /> <origin xyz="0.0 0.0 0.0" rpy="0.0 0.0 0.0" />
+        <child link="base_link" />
+        <origin xyz="0.0 0.0 0.0" rpy="0.0 0.0 0.0" />
     </joint>
     <link name="pestle">
@@ -15,4 +16,7 @@
                 <mesh filename="package://ros_study/meshes/pestle_ur.stl" />
             </geometry>
+            <material name="LightGrey">
+                <color rgba="0.7 0.7 0.7 1.0"/>
+            </material>
         </visual>
         <collision>
@@ -25,5 +29,6 @@
     <joint name="joint_pestle" type="fixed">
         <origin rpy="0 0 0" xyz="0 0 0" />
-        <parent link="tool0" /> <child link="pestle" />
+        <parent link="tool0" />
+        <child link="pestle" />
     </joint>
     <link name="pestle_tip" />
@@ -39,4 +44,5 @@
                 <mesh filename="package://ros_study/meshes/spatula.stl" />
             </geometry>
+            <material name="LightGrey"/>
         </visual>
         <collision>
@@ -49,5 +55,6 @@
     <joint name="joint_spatula" type="fixed">
         <origin rpy="0 ${-pi/2} 0" xyz="-0.03655 0 0.0135" />
-        <parent link="tool0" /> <child link="spatula" />
+        <parent link="tool0" />
+        <child link="spatula" />
     </joint>
     <link name="spatula_tip" />
@@ -60,5 +67,6 @@
     <joint name="joint_dummy_ee" type="fixed">
         <origin rpy="0 0 0" xyz="0 0 0" />
-        <parent link="tool0" /> <child link="dummy_ee" />
+        <parent link="tool0" />
+        <child link="dummy_ee" />
     </joint>
 </robot>
