Commit message: Update

File: slides/ros-simulator-connection/code/ros2/ur5e_with_eef_add_controller.xacro (robot description, xacro)
@@ -4,4 +4,10 @@
     <xacro:arg name="pestle_length" default="0.1092" />
     <xacro:arg name="spatula_length" default="0.089" />
+    <link name="world" />
+    <joint name="world_joint" type="fixed">
+        <parent link="world" />
+        <child link="base_link" />
+        <origin xyz="0.0 0.0 0.0" rpy="0.0 0.0 0.0" />
+    </joint>
     <link name="pestle">
         <visual>
