Commit message: Add ros controll mock system

File: slides/ros-simulator-connection/code/ros2/ur5e_with_ee.xacro (robot description, xacro)
@@ -10,4 +10,39 @@
         <origin xyz="0.0 0.0 0.0" rpy="0.0 0.0 0.0" />
     </joint>
+    <ros2_control name="UR5eMockSystem" type="system">
+        <hardware>
+            <plugin>mock_components/GenericSystem</plugin>
+        </hardware>
+        <joint name="shoulder_pan_joint">
+            <command_interface name="position" />
+            <state_interface name="position"><param name="initial_value">0.0</param></state_interface>
+            <state_interface name="velocity"/>
+        </joint>
+        <joint name="shoulder_lift_joint">
+            <command_interface name="position" />
+            <state_interface name="position"><param name="initial_value">-1.57</param></state_interface>
+            <state_interface name="velocity"/>
+        </joint>
+        <joint name="elbow_joint">
+            <command_interface name="position" />
+            <state_interface name="position"><param name="initial_value">0.0</param></state_interface>
+            <state_interface name="velocity"/>
+        </joint>
+        <joint name="wrist_1_joint">
+            <command_interface name="position" />
+            <state_interface name="position"><param name="initial_value">-1.57</param></state_interface>
+            <state_interface name="velocity"/>
+        </joint>
+        <joint name="wrist_2_joint">
+            <command_interface name="position" />
+            <state_interface name="position"><param name="initial_value">0.0</param></state_interface>
+            <state_interface name="velocity"/>
+        </joint>
+        <joint name="wrist_3_joint">
+            <command_interface name="position" />
+            <state_interface name="position"><param name="initial_value">0.0</param></state_interface>
+            <state_interface name="velocity"/>
+        </joint>
+    </ros2_control>
     <link name="pestle">
         <visual>
@@ -70,3 +105,3 @@
         <child link="dummy_ee" />
     </joint>
-</robot>
+    </robot>
