Commit message: rearange package

File: ros2_ws/src/ros_study/urdf/ur5e_with_ee.xacro (robot description, xacro)
@@ -34,5 +34,5 @@
            <origin xyz="0 0 0.0001" rpy="0 0 0" />
            <geometry>
-               <mesh filename="package://ros_study_description/meshes/pestle_ur.stl" />
+               <mesh filename="package://ros_study/meshes/pestle_ur.stl" />
            </geometry>
            <material name="LightGrey">
@@ -43,5 +43,5 @@
            <origin xyz="0 0 0.0001" rpy="0 0 0" />
            <geometry>
-               <mesh filename="package://ros_study_description/meshes/pestle_ur.stl" />
+               <mesh filename="package://ros_study/meshes/pestle_ur.stl" />
            </geometry>
        </collision>
@@ -62,5 +62,5 @@
            <origin xyz="0 0 0.0001" rpy="0 0 0" />
            <geometry>
-               <mesh filename="package://ros_study_description/meshes/spatula.stl" />
+               <mesh filename="package://ros_study/meshes/spatula.stl" />
            </geometry>
            <material name="LightGrey"/>
@@ -69,5 +69,5 @@
            <origin xyz="0 0 0.0001" rpy="0 0 0" />
            <geometry>
-               <mesh filename="package://ros_study_description/meshes/spatula.stl" />
+               <mesh filename="package://ros_study/meshes/spatula.stl" />
            </geometry>
        </collision>

File: ros2_ws/src/ros_study/urdf/ur5e_with_ee_gazebo.xacro (robot description, xacro)
@@ -1,5 +1,5 @@
 <?xml version="1.0"?>
 <robot xmlns:xacro="http://www.ros.org/wiki/xacro" name="ur">
-    <xacro:include filename="$(find ros_study_description)/urdf/ur5e.xacro" />
+    <xacro:include filename="$(find ros_study)/urdf/ur5e.xacro" />
     <xacro:arg name="controllers_file" default="" />
     <xacro:arg name="pestle_length" default="0.1092" />
@@ -50,5 +50,5 @@
             <origin xyz="0 0 0.0001" rpy="0 0 0" />
             <geometry>
-                <mesh filename="package://ros_study_description/meshes/pestle_ur.stl" />
+                <mesh filename="package://ros_study/meshes/pestle_ur.stl" />
             </geometry>
             <material name="LightGrey">
@@ -59,5 +59,5 @@
             <origin xyz="0 0 0.0001" rpy="0 0 0" />
             <geometry>
-                <mesh filename="package://ros_study_description/meshes/pestle_ur.stl" />
+                <mesh filename="package://ros_study/meshes/pestle_ur.stl" />
             </geometry>
         </collision>
@@ -78,5 +78,5 @@
             <origin xyz="0 0 0.0001" rpy="0 0 0" />
             <geometry>
-                <mesh filename="package://ros_study_description/meshes/spatula.stl" />
+                <mesh filename="package://ros_study/meshes/spatula.stl" />
             </geometry>
             <material name="LightGrey" />
@@ -85,5 +85,5 @@
             <origin xyz="0 0 0.0001" rpy="0 0 0" />
             <geometry>
-                <mesh filename="package://ros_study_description/meshes/spatula.stl" />
+                <mesh filename="package://ros_study/meshes/spatula.stl" />
             </geometry>
         </collision>

File: ros2_ws/src/ros_study/urdf/ur5e_with_ee_mock_components.xacro (robot description, xacro)
@@ -1,5 +1,5 @@
 <?xml version="1.0"?>
 <robot xmlns:xacro="http://www.ros.org/wiki/xacro" name="ur">
-    <xacro:include filename="$(find ros_study_description)/urdf/ur5e.xacro" />
+    <xacro:include filename="$(find ros_study)/urdf/ur5e.xacro" />
     <xacro:arg name="pestle_length" default="0.1092" />
     <xacro:arg name="spatula_length" default="0.089" />
@@ -49,5 +49,5 @@
             <origin xyz="0 0 0.0001" rpy="0 0 0" />
             <geometry>
-                <mesh filename="package://ros_study_description/meshes/pestle_ur.stl" />
+                <mesh filename="package://ros_study/meshes/pestle_ur.stl" />
             </geometry>
             <material name="LightGrey">
@@ -58,5 +58,5 @@
             <origin xyz="0 0 0.0001" rpy="0 0 0" />
             <geometry>
-                <mesh filename="package://ros_study_description/meshes/pestle_ur.stl" />
+                <mesh filename="package://ros_study/meshes/pestle_ur.stl" />
             </geometry>
         </collision>
@@ -77,5 +77,5 @@
             <origin xyz="0 0 0.0001" rpy="0 0 0" />
             <geometry>
-                <mesh filename="package://ros_study_description/meshes/spatula.stl" />
+                <mesh filename="package://ros_study/meshes/spatula.stl" />
             </geometry>
             <material name="LightGrey" />
@@ -84,5 +84,5 @@
             <origin xyz="0 0 0.0001" rpy="0 0 0" />
             <geometry>
-                <mesh filename="package://ros_study_description/meshes/spatula.stl" />
+                <mesh filename="package://ros_study/meshes/spatula.stl" />
             </geometry>
         </collision>
