Commit message: fix bug

File: ros2_ws/src/ros_study/urdf/ur5e_with_ee_for_real_robot.xacro (robot description, xacro)
@@ -2,14 +2,32 @@
 <robot xmlns:xacro="http://wiki.ros.org/xacro" name="ur">
    <xacro:arg name="name" default="ur"/>
+   <xacro:arg name="ur_type" default="ur5e"/>
    <xacro:arg name="tf_prefix" default="" />
+   <xacro:arg name="use_fake_hardware" default="true"/>
+   <xacro:arg name="fake_sensor_commands" default="true"/>
+   <xacro:arg name="robot_ip" default="0.0.0.0"/>
+   <xacro:arg name="script_filename" default=""/>
+   <xacro:arg name="output_recipe_filename" default=""/>
+   <xacro:arg name="input_recipe_filename" default=""/>
    <xacro:arg name="pestle_length" default="0.1092" />
    <xacro:arg name="spatula_length" default="0.089" />
-   <xacro:include filename="$(find ros_study)/urdf/ur5e.xacro"/>
+   <xacro:include filename="$(find ur_description)/urdf/ur_macro.xacro"/>
+   <xacro:ur_robot
+     name="$(arg name)"
+     tf_prefix="$(arg tf_prefix)"
+     parent="world"
+     joint_limits_parameters_file="$(find ur_description)/config/$(arg ur_type)/joint_limits.yaml"
+     kinematics_parameters_file="$(find ur_description)/config/$(arg ur_type)/default_kinematics.yaml"
+     physical_parameters_file="$(find ur_description)/config/$(arg ur_type)/physical_parameters.yaml"
+     visual_parameters_file="$(find ur_description)/config/$(arg ur_type)/visual_parameters.yaml"
+     use_fake_hardware="$(arg use_fake_hardware)"
+     fake_sensor_commands="$(arg fake_sensor_commands)"
+     robot_ip="$(arg robot_ip)"
+     script_filename="$(arg script_filename)"
+     output_recipe_filename="$(arg output_recipe_filename)"
+     input_recipe_filename="$(arg input_recipe_filename)">
+     <origin xyz="0 0 0" rpy="0 0 0" />
+   </xacro:ur_robot>
    <link name="world" />
-   <joint name="world_joint" type="fixed">
-       <origin xyz="0 0 0" rpy="0 0 0" />
-       <parent link="world" />
-       <child link="base_link" />
-   </joint>
    <link name="pestle">
        <visual>

File: ros2_ws/src/ros_study/urdf/ur5e_with_ee_mock_components.xacro (robot description, xacro)
@@ -1,12 +1,14 @@
 <?xml version="1.0"?>
-<robot xmlns:xacro="http://www.ros.org/wiki/xacro" name="ur">
-    <xacro:include filename="$(find ros_study)/urdf/ur5e.xacro" />
+<robot xmlns:xacro="http://wiki.ros.org/xacro" name="ur">
+    <xacro:arg name="name" default="ur"/>
+    <xacro:arg name="tf_prefix" default="" />
     <xacro:arg name="pestle_length" default="0.1092" />
     <xacro:arg name="spatula_length" default="0.089" />
+    <xacro:include filename="$(find ros_study)/urdf/ur5e.xacro" />
     <link name="world" />
     <joint name="world_joint" type="fixed">
+        <origin xyz="0 0 0" rpy="0 0 0" />
         <parent link="world" />
         <child link="base_link" />
-        <origin xyz="0.0 0.0 0.0" rpy="0.0 0.0 0.0" />
     </joint>
     <ros2_control name="UR5eMockSystem" type="system">
@@ -16,30 +18,42 @@
         <joint name="shoulder_pan_joint">
             <command_interface name="position" />
-            <state_interface name="position"><param name="initial_value">0.0</param></state_interface>
+            <state_interface name="position">
+                <param name="initial_value">0.0</param>
+            </state_interface>
             <state_interface name="velocity" />
         </joint>
         <joint name="shoulder_lift_joint">
             <command_interface name="position" />
-            <state_interface name="position"><param name="initial_value">-1.57</param></state_interface>
+            <state_interface name="position">
+                <param name="initial_value">-1.57</param>
+            </state_interface>
             <state_interface name="velocity" />
         </joint>
         <joint name="elbow_joint">
             <command_interface name="position" />
-            <state_interface name="position"><param name="initial_value">0.0</param></state_interface>
+            <state_interface name="position">
+                <param name="initial_value">0.0</param>
+            </state_interface>
             <state_interface name="velocity" />
         </joint>
         <joint name="wrist_1_joint">
             <command_interface name="position" />
-            <state_interface name="position"><param name="initial_value">-1.57</param></state_interface>
+            <state_interface name="position">
+                <param name="initial_value">-1.57</param>
+            </state_interface>
             <state_interface name="velocity" />
         </joint>
         <joint name="wrist_2_joint">
             <command_interface name="position" />
-            <state_interface name="position"><param name="initial_value">0.0</param></state_interface>
+            <state_interface name="position">
+                <param name="initial_value">0.0</param>
+            </state_interface>
             <state_interface name="velocity" />
         </joint>
         <joint name="wrist_3_joint">
             <command_interface name="position" />
-            <state_interface name="position"><param name="initial_value">0.0</param></state_interface>
+            <state_interface name="position">
+                <param name="initial_value">0.0</param>
+            </state_interface>
             <state_interface name="velocity" />
         </joint>
@@ -52,5 +66,5 @@
             </geometry>
             <material name="LightGrey">
-                <color rgba="0.7 0.7 0.7 1.0" />
+                <color rgba="0.7 0.7 0.7 1.0"/>
             </material>
         </visual>
@@ -79,5 +93,5 @@
                 <mesh filename="package://ros_study/meshes/spatula.stl" />
             </geometry>
-            <material name="LightGrey" />
+            <material name="LightGrey"/>
         </visual>
         <collision>
